File: usb_board/usb_board.kicad_pcb (KiCad board)
At the start: 2 copper layers, 50 x 25 mm, 13 parts, among them J1 IN_5V, J2 IN_5V, J3 USB_A, J4 USB_A, J5 USB_A

Commit message: update usb board
Parts:
- removed REF** (x4): MountingHole_3.2mm_M3_Pad, MountingHole:MountingHole_3.2mm_M3_Pad
- added R2: 10k, Resistor_SMD:R_0805_2012Metric_Pad1.15x1.40mm_HandSolder, B.Cu at (181.5, 107.0)
- added R3: 10k, Resistor_SMD:R_0805_2012Metric_Pad1.15x1.40mm_HandSolder, B.Cu at (181.5, 102.0)
- added R4: 10k, Resistor_SMD:R_0805_2012Metric_Pad1.15x1.40mm_HandSolder, B.Cu at (191.5, 107.0)
- added R5: 10k, Resistor_SMD:R_0805_2012Metric_Pad1.15x1.40mm_HandSolder, B.Cu at (191.5, 102.0)
- added R6: 10k, Resistor_SMD:R_0805_2012Metric_Pad1.15x1.40mm_HandSolder, B.Cu at (201.5, 107.0)
- added R7: 10k, Resistor_SMD:R_0805_2012Metric_Pad1.15x1.40mm_HandSolder, B.Cu at (201.5, 102.0)
Connections:
- J3 pad 3: Net-(J3-Pad3) -> Net-(J3-Pad2)
- J4 pad 3: Net-(J4-Pad3) -> Net-(J4-Pad2)
- J5 pad 3: Net-(J5-Pad3) -> Net-(J5-Pad2)
Routing:
- net GND: track 0.00 -> 7.53 mm
- net +5V: track 2.51 -> 10.0 mm
- net Net-(J5-Pad2): track 0.00 -> 7.39 mm
- net Net-(J4-Pad2): track 0.00 -> 7.39 mm
- net Net-(J3-Pad2): track 0.00 -> 7.38 mm
Other:
- board text added: "+5V"
- board text added: "GND"
